File: pcb/ortho40.kicad_sch (KiCad schematic)
At the start: 129 parts, among them J1 SWD, J2 USB_C_Receptacle_USB2.0, SW1 SW_Push, U1 RP2040, U2 XC6206PxxxMR, U3 W25Q128JVS, U4 USBLC6-2SC6, U5 ST7735S_1.8inch, Y1 12MHz

Commit message: More changes...
Parts:
- C1: footprint Capacitor_SMD:C_0402_1005Metric -> MountingHole:MountingHole_2.2mm_M2
- renumbered MX8 to MX10, MX10 to MX11, MX15 to MX14, MX14 to MX15, MX19 to MX18, MX21 to MX19, MX3 to MX2, MX23 to MX20, MX18 to MX21, MX20 to MX22, MX22 to MX23, MX27 to MX26, MX26 to MX27, MX2 to MX3, MX31 to MX30, MX33 to MX31, MX35 to MX32, MX30 to MX33, MX32 to MX34, MX34 to MX35, MX39 to MX38, MX38 to MX39, MX43 to MX42, MX45 to MX43, MX47 to MX44, MX42 to MX45, MX44 to MX46, MX46 to MX47, MX7 to MX6, MX9 to MX7, MX11 to MX8, MX6 to MX9

Commit message: Use the correct footprint for the display
Parts:
- added C7: 10uF, Capacitor_SMD:C_0402_1005Metric, symbol Device:C_Small
- C1: footprint MountingHole:MountingHole_2.2mm_M2 -> Capacitor_SMD:C_0402_1005Metric
- SW1: footprint Connector_PinHeader_2.54mm:PinHeader_1x02_P2.54mm_Vertical -> Button_Switch_SMD:SW_SPST_CK_KXT3
- U5: footprint Footprints:ST7735_1.8inch -> Footprints:DFR0928
- renumbered C9 to C10, C10 to C11, C11 to C12, C12 to C13, C13 to C14, C14 to C15, C15 to C16, C16 to C17, C7 to C8, C8 to C9
Connections:
- net +3V3: now also C7.1
- net GND: now also C7.2
- no-connect marks 3 -> 2
Other:
- moved on the sheet: C10, C11, C12, C13, C14, C15, C4, C5, C6, C8, C9

Commit message: Finishing touches for rev 2
Parts:
- SW1: value SW_Push -> BOOTSEL; footprint Button_Switch_SMD:SW_SPST_CK_KXT3 -> Button_Switch_SMD:SW_Push_SPST_NO_Alps_SKRK
Changed lines of the file:
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@@
     (in_bom yes) (on_board yes) (fields_autoplaced)
     (property "Reference" "SW1" (id 0) (at 132.588 115.57 0))
-    (property "Value" "SW_Push" (id 1) (at 132.588 118.11 0))
-    (property "Footprint" "Button_Switch_SMD:SW_SPST_CK_KXT3" (id 2) (at 132.588 118.364 0)
+    (property "Value" "BOOTSEL" (id 1) (at 132.588 118.11 0))
+    (property "Footprint" "Button_Switch_SMD:SW_Push_SPST_NO_Alps_SKRK" (id 2) (at 132.588 118.364 0)
       (effects (font (size 1.27 1.27)) hide)
     )
@@
     )
     (path "/f037e8ae-b9e9-4cd6-86ad-07d55b362385"
-      (reference "SW1") (unit 1) (value "SW_Push") (footprint "Button_Switch_SMD:SW_SPST_CK_KXT3")
+      (reference "SW1") (unit 1) (value "BOOTSEL") (footprint "Button_Switch_SMD:SW_Push_SPST_NO_Alps_SKRK")
     )
     (path "/912c4917-ada4-4990-9da6-1eac395cf218"
